Commit message: Automatic update of urdf triggered by GitHub Action
ergocub-software = 05614341d63ddf640d4cdb0748f8975cde6ea481
cad-libraries    = https://github.com/icub-tech-iit/cad-libraries/commit/c4929f014c3aeab36398a9daafee3e78af25539c
cad-mechanics    = https://github.com/icub-tech-iit/cad-mechanics/commit/f83508ec601e65b08c3dc15d2f198bab48901569
creo2urdf        = https://github.com/icub-tech-iit/creo2urdf/releases/tag/v0.5.18

File: urdf/ergoCub/robots/ergoCubGazeboSN000/model.urdf (robot description, URDF)
Before this commit: robot ergoCub, 204 links, 203 joints
Links:
- removed link chest
- removed link neck_2
- removed link neck_3
- added link SIM_ECUB_1-1_CHEST, mass 8.065471632648594; collision mesh filename=package://ergoCub/meshes/simmechanics/sim_ecub_1-1_chest.stl scale=0.001 0.001 0.001; visual mesh filename=package://ergoCub/meshes/simmechanics/sim_ecub_1-1_chest.stl scale=0.001 0.001 0.001
- added link SIM_ECUB_1-1_HEAD_NECK_2, mass 0.12100314943032965; collision mesh filename=package://ergoCub/meshes/simmechanics/sim_ecub_1-1_head_nec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 scale=0.001 0.001 0.001; visual mesh filename=package://ergoCub/meshes/simmechanics/sim_ecub_1-1_head_nec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 scale=0.001 0.001 0.001
- added link SIM_ECUB_1-1_HEAD_NECK_3, mass 0.17811376821431446; collision mesh filename=package://ergoCub/meshes/simmechanics/sim_ecub_1-1_head_nec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 scale=0.001 0.001 0.001; visual mesh filename=package://ergoCub/meshes/simmechanics/sim_ecub_1-1_head_nec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 scale=0.001 0.001 0.001
- link head: geometry collision mesh filename=package://ergoCub/meshes/simmechanics/sim_ecub_1-1_head.stl scale=0.001 0.001 0.001; visual mesh filename=package://ergoCub/meshes/simmechanics/sim_ecub_1-1_head.stl scale=0.001 0.001 0.001
Joints:
- removed joint l_shoulder_pitch
- removed joint neck_pitch
- removed joint neck_roll
- removed joint neck_yaw
- removed joint r_shoulder_pitch
- removed joint torso_yaw
- added joint SIM_ECUB_1-1_CHEST--SIM_ECUB_1-1_HEAD_NECK_2: type continuous, parent SIM_ECUB_1-1_CHEST, child SIM_ECUB_1-1_HEAD_NECK_2, origin xyz=1.2708867293726507e-15 -0.004861512347971573 0.28976999999999997 rpy=-1.3208254231267427e-15 8.743006792683972e-16 1.634109514370152e-15, axis 1 -3.0212645743512393e-15 -4.235220117208732e-15
- added joint SIM_ECUB_1-1_CHEST--SIM_ECUB_1-1_L_SHOULDER_1: type continuous, parent SIM_ECUB_1-1_CHEST, child l_shoulder_1, origin xyz=0.06704761117227556 0.01351867684261036 0.18798981080941732 rpy=0.25361232387325056 -0.05203160550449709 -1.8460750592087682, axis 1.0928757898653885e-16 1 3.0531133177191805e-16
- added joint SIM_ECUB_1-1_CHEST--SIM_ECUB_1-1_R_SHOULDER_1: type continuous, parent SIM_ECUB_1-1_CHEST, child r_shoulder_1, origin xyz=-0.06704761117227384 0.013518676842610497 0.18798981080941812 rpy=-0.25361232387326527 -0.05203160550449503 -1.2955175943810264, axis 6.574601973952099e-16 -1.0000000000000004 -3.3029134982598407e-15
- added joint SIM_ECUB_1-1_HEAD_NECK_2--SIM_ECUB_1-1_HEAD_NECK_3: type continuous, parent SIM_ECUB_1-1_HEAD_NECK_2, child SIM_ECUB_1-1_HEAD_NECK_3, origin xyz=2.83678257316353e-16 0.004861512347971555 0.009499999999999842 rpy=2.1824457611556613e-31 -6.353369076823475e-18 -2.0572736222891147e-18, axis 1.4901274658640806e-15 1 -1.270579771067814e-31
- added joint SIM_ECUB_1-1_HEAD_NECK_3--SIM_ECUB_1-1_HEAD: type continuous, parent SIM_ECUB_1-1_HEAD_NECK_3, child head, origin xyz=4.2173434983493643e-16 -0.004861512347971283 0.06914999999999982 rpy=-5.890991943503742e-15 -4.922977909666296e-15 -1.5707963267948977, axis 1.408209052907529e-15 5.709519748275234e-16 0.9999999999999997
- added joint SIM_ECUB_1-1_TORSO_2--SIM_ECUB_1-1_CHEST: type continuous, parent torso_2, child SIM_ECUB_1-1_CHEST, origin xyz=3.2264224928916605e-18 1.297606021580521e-16 3.795334199281987e-17 rpy=1.4239886692466165e-15 -6.938893903909127e-18 1.5707963267948966, axis -6.092934465537603e-15 -3.5088530983238434e-15 -1
- joint camera_tilt: axis 1.9074075506529947e-16 -1 -1.4146048262463281e-15 -> 1.1750855152298039e-16 -1 -2.1665209362190277e-15
- joint l_ankle_pitch: axis -2.389602037081462e-16 1 1.4538275231733847e-16 -> -2.38960203708147e-16 1 1.4538275231733847e-16
- joint l_ankle_roll: axis 1 -4.05028482201375e-16 -1.2496691978128869e-15 -> 1 -4.050284822013754e-16 -1.2496691978128869e-15
- joint l_elbow: axis -8.847089727469744e-17 -0.9999999999999953 6.383782391594399e-15 -> -2.550043509679755e-16 -0.999999999999986 1.293409823688246e-14
- joint l_hip_pitch: axis -5.772831379991284e-17 -1 -1.3843833381666392e-17 -> -5.772831379991284e-17 -1 -1.384383338166718e-17
- joint l_hip_roll: axis 1 -6.123233995736708e-17 6.3201403498236e-16 -> 1 -6.123233995736708e-17 6.320140349823599e-16
- joint l_hip_yaw: axis -8.622588011769357e-16 1.5936665473077025e-16 1 -> -8.622588011769357e-16 1.5936665473077023e-16 1
- joint l_index_add: axis -3.232245792329867e-15 -0.9999999999999998 1.5397182495276352e-15 -> -3.3702260559116687e-15 -0.9999999999999993 1.0014973022447945e-15
- joint l_index_dist: axis -0.9999999999999997 1.2698175844150033e-15 1.3045120539345794e-15 -> -0.999999999999999 1.1587952819524896e-15 1.3045120539345763e-15
- joint l_index_prox: axis -0.9999999999999996 -2.0816681711721439e-16 3.99680288865056e-15 -> -0.9999999999999987 -3.1918911957972767e-16 4.024558464266183e-15
- joint l_knee: axis -2.608937546411318e-16 -1 5.166588955193111e-17 -> -2.60893754641131e-16 -1 5.166588955193113e-17
- joint l_middle_dist: axis -0.9999999999999998 -2.3467059288222403e-15 6.408211626924537e-16 -> -0.9999999999999993 -2.3467707837629264e-15 5.921449210147216e-16
- joint l_middle_prox: axis -0.9999999999999998 -1.0130785099575306e-15 -4.37150315993994e-16 -> -0.9999999999999993 -1.0685896612017132e-15 -4.78783679465276e-16
- joint l_pinkie_dist: axis -1.0000000000000002 -2.6194156222657784e-15 3.3662023329484224e-16 -> -1.0000000000000007 -2.6471672680994334e-15 3.0885679776748995e-16
- joint l_pinkie_prox: axis -1.0000000000000002 -1.1843525269243981e-15 5.273559366969494e-16 -> -1.0000000000000004 -1.1774136330204909e-15 4.996003610813204e-16
- joint l_ring_dist: axis -1.0000000000000002 -2.168404344970969e-17 1.2490009027033007e-15 -> -1.0000000000000007 -1.3270634591222456e-16 1.2351231148954863e-15
- joint l_ring_prox: axis -1.0000000000000002 -1.0100531863796072e-15 6.800116025829084e-16 -> -1.0000000000000004 -1.055155996755004e-15 6.522560269672795e-16
- joint l_shoulder_roll: axis 1 3.78169717762985e-16 2.7478019859473113e-15 -> 1 3.226585665316948e-16 2.775557561563002e-15
- joint l_shoulder_yaw: axis -3.00454106039183e-14 2.9143354396410367e-15 -0.9999999999999978 -> -6.00908212078363e-14 6.050715484207078e-15 -0.9999999999999933
- joint l_thumb_add: axis 3.3306690738754696e-16 -6.245004513516506e-16 -0.9999999999999998 -> 4.996003610813204e-16 -1.124100812432971e-15 -0.9999999999999993
- joint l_thumb_dist: axis -1.4016565559607482e-15 4.996003048844505e-16 -1 -> -1.901256909464961e-15 1.1102229532740747e-15 -1
- joint l_thumb_prox: axis 9.575673587391975e-16 -1.4988010832439613e-15 -1.0000000000000002 -> 4.163336342344337e-16 -9.992007221626409e-16 -1.0000000000000004
- joint l_wrist_pitch: axis -7.632783294297949e-17 -0.9999999999999999 -4.163336342344336e-16 -> -1.8735013540549497e-16 -0.9999999999999997 -1.0269562977782694e-15
- joint l_wrist_roll: axis -0.9999999999999999 4.805184028455756e-16 1.3877787807814474e-16 -> -0.9999999999999997 6.47051856539349e-16 7.632783294297998e-17
- joint l_wrist_yaw: axis -2.994132719535971e-14 2.9420910152566727e-15 -0.9999999999999982 -> -6.005612673831686e-14 5.828670879282063e-15 -0.9999999999999947
- joint r_ankle_pitch: axis -3.505264366441263e-17 1 -1.331317022347139e-16 -> -3.505264366441327e-17 1 -1.3313170223472496e-16
- joint r_ankle_roll: axis -1 -1.628246671334752e-16 2.560295622560413e-15 -> -1 -1.628246671334752e-16 2.5602956225604195e-15
- joint r_elbow: axis 2.4459601011270737e-16 -1.0000000000000027 1.2989609388114332e-14 -> 3.5561831257529417e-16 -1.000000000000008 2.5951463200613154e-14
- joint r_hip_pitch: axis -1.0880513989386065e-16 -1 1.384383338166008e-17 -> -1.0880513989386065e-16 -1 1.3843833381659292e-17
- joint r_hip_roll: axis -1 -3.3813287685016297e-16 -7.120227705451219e-17 -> -1 -3.3813287685016258e-16 -7.12022770545114e-17
- joint r_hip_yaw: axis -2.395305022015389e-20 1.474932849181089e-15 -1 -> -2.3953050200826797e-20 1.474932849181089e-15 -1
- joint r_index_add: axis -2.2710721778544278e-14 1.0000000000000058 -3.325533406549057e-15 -> -4.651242255183732e-14 1.0000000000000173 -6.08487548946725e-15
- joint r_index_dist: axis -1.0000000000000127 4.898859096158517e-14 -3.955169525227743e-16 -> -1.000000000000038 9.6672669869238e-14 -5.134781488895157e-16
- joint r_index_prox: axis -1.0000000000000127 4.871797409933279e-14 5.689893001203353e-16 -> -1.000000000000038 9.645756415821688e-14 3.8163916471455337e-16
- joint r_knee: axis 1.2193157766326317e-6 -0.9999999999992567 4.719551160658935e-15 -> 1.219315776632632e-6 -0.9999999999992569 4.719551160658948e-15
- joint r_middle_dist: axis -1.0000000000000127 4.8869412818017636e-14 7.711215903793126e-16 -> -1.000000000000038 9.694733146028018e-14 8.607486116259909e-16
- joint r_middle_prox: axis -1.0000000000000067 2.2546201017270685e-14 -2.45636844198318e-15 -> -1.00000000000002 4.66935518028684e-14 -2.470246229791037e-15
- joint r_pinkie_dist: axis -1.0000000000000142 4.6843605383539805e-14 1.91513471747844e-15 -> -1.0000000000000426 9.46109510180395e-14 2.164934898019344e-15
- joint r_pinkie_prox: axis -1.0000000000000073 2.687697787657948e-14 -2.761679773755077e-15 -> -1.0000000000000224 5.074677290602035e-14 -2.581268532253489e-15
- joint r_ring_dist: axis -1.0000000000000142 4.792260338559737e-14 -2.890049310977331e-15 -> -1.0000000000000426 9.566219344448145e-14 -2.647188024340446e-15
- joint r_ring_prox: axis -1.0000000000000073 2.7031320490650422e-14 -2.5396351688300456e-15 -> -1.0000000000000222 5.091846275485106e-14 -2.345346139520643e-15
- joint r_shoulder_roll: axis -1.0000000000000009 8.205242041369425e-16 1.734723475977312e-16 -> -1.0000000000000027 1.153591111524405e-15 1.9428902930949706e-16
- joint r_shoulder_yaw: axis -4.579669976578765e-16 5.551115123125817e-17 1 -> -4.371503159461546e-16 8.32667268468839e-17 1
- joint r_thumb_add: axis 1.304512053934559e-15 4.801714581503802e-15 1.0000000000000062 -> 3.3584246494910985e-15 1.0560996521746802e-14 1.0000000000000187
- joint r_thumb_dist: axis -5.290212712338784e-14 -2.997602166487913e-14 -1.0000000000000502 -> -1.5804024755539139e-13 -8.88733531212472e-14 -1.0000000000001505
- joint r_thumb_prox: axis -3.549938121238938e-14 -1.840194663316197e-14 -1.0000000000000255 -> -7.101264021258658e-14 -3.7719827261639693e-14 -1.0000000000000764
- joint r_wrist_pitch: axis 5.100087019371814e-16 -1 -5.273559366969494e-16 -> 4.544975507059239e-16 -1 -1.1379786002407858e-15
- joint r_wrist_roll: axis 1.0000000000000004 -1.8735013540549512e-16 7.632783294297946e-17 -> 1.0000000000000013 -2.42861286636753e-16 4.857225732735043e-17
- joint r_wrist_yaw: axis 5.7037707890117685e-15 -1.2517764602648659e-14 1.0000000000000022 -> 1.1289580381657174e-14 -2.514655150775995e-14 1.0000000000000067
- joint torso_pitch: axis 1.9259299443837326e-34 1 0 -> 3.851859888763962e-34 1 0

File: urdf/ergoCub/robots/ergoCubGazeboSN000_minContacts/model.urdf (robot description, URDF)
Before this commit: robot ergoCub, 204 links, 203 joints
Links:
- removed link chest
- removed link neck_2
- removed link neck_3
- added link SIM_ECUB_1-1_CHEST, mass 8.065471632648594; collision mesh filename=package://ergoCub/meshes/simmechanics/sim_ecub_1-1_chest.stl scale=0.001 0.001 0.001; visual mesh filename=package://ergoCub/meshes/simmechanics/sim_ecub_1-1_chest.stl scale=0.001 0.001 0.001
- added link SIM_ECUB_1-1_HEAD_NECK_2, mass 0.12100314943032965; collision mesh filename=package://ergoCub/meshes/simmechanics/sim_ecub_1-1_head_nec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 scale=0.001 0.001 0.001; visual mesh filename=package://ergoCub/meshes/simmechanics/sim_ecub_1-1_head_nec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 scale=0.001 0.001 0.001
- added link SIM_ECUB_1-1_HEAD_NECK_3, mass 0.17811376821431446; collision mesh filename=package://ergoCub/meshes/simmechanics/sim_ecub_1-1_head_nec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 scale=0.001 0.001 0.001; visual mesh filename=package://ergoCub/meshes/simmechanics/sim_ecub_1-1_head_nec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 scale=0.001 0.001 0.001
- link head: geometry visual mesh filename=package://ergoCub/meshes/simmechanics/sim_ecub_1-1_head.stl scale=0.001 0.001 0.001
Joints:
- removed joint l_shoulder_pitch
- removed joint neck_pitch
- removed joint neck_roll
- removed joint neck_yaw
- removed joint r_shoulder_pitch
- removed joint torso_yaw
- added joint SIM_ECUB_1-1_CHEST--SIM_ECUB_1-1_HEAD_NECK_2: type continuous, parent SIM_ECUB_1-1_CHEST, child SIM_ECUB_1-1_HEAD_NECK_2, origin xyz=1.2708867293726507e-15 -0.004861512347971573 0.28976999999999997 rpy=-1.3208254231267427e-15 8.743006792683972e-16 1.634109514370152e-15, axis 1 -3.0212645743512393e-15 -4.235220117208732e-15
- added joint SIM_ECUB_1-1_CHEST--SIM_ECUB_1-1_L_SHOULDER_1: type continuous, parent SIM_ECUB_1-1_CHEST, child l_shoulder_1, origin xyz=0.06704761117227556 0.01351867684261036 0.18798981080941732 rpy=0.25361232387325056 -0.05203160550449709 -1.8460750592087682, axis 1.0928757898653885e-16 1 3.0531133177191805e-16
- added joint SIM_ECUB_1-1_CHEST--SIM_ECUB_1-1_R_SHOULDER_1: type continuous, parent SIM_ECUB_1-1_CHEST, child r_shoulder_1, origin xyz=-0.06704761117227384 0.013518676842610497 0.18798981080941812 rpy=-0.25361232387326527 -0.05203160550449503 -1.2955175943810264, axis 6.574601973952099e-16 -1.0000000000000004 -3.3029134982598407e-15
- added joint SIM_ECUB_1-1_HEAD_NECK_2--SIM_ECUB_1-1_HEAD_NECK_3: type continuous, parent SIM_ECUB_1-1_HEAD_NECK_2, child SIM_ECUB_1-1_HEAD_NECK_3, origin xyz=2.83678257316353e-16 0.004861512347971555 0.009499999999999842 rpy=2.1824457611556613e-31 -6.353369076823475e-18 -2.0572736222891147e-18, axis 1.4901274658640806e-15 1 -1.270579771067814e-31
- added joint SIM_ECUB_1-1_HEAD_NECK_3--SIM_ECUB_1-1_HEAD: type continuous, parent SIM_ECUB_1-1_HEAD_NECK_3, child head, origin xyz=4.2173434983493643e-16 -0.004861512347971283 0.06914999999999982 rpy=-5.890991943503742e-15 -4.922977909666296e-15 -1.5707963267948977, axis 1.408209052907529e-15 5.709519748275234e-16 0.9999999999999997
- added joint SIM_ECUB_1-1_TORSO_2--SIM_ECUB_1-1_CHEST: type continuous, parent torso_2, child SIM_ECUB_1-1_CHEST, origin xyz=3.2264224928916605e-18 1.297606021580521e-16 3.795334199281987e-17 rpy=1.4239886692466165e-15 -6.938893903909127e-18 1.5707963267948966, axis -6.092934465537603e-15 -3.5088530983238434e-15 -1
- joint camera_tilt: axis 1.9074075506529947e-16 -1 -1.4146048262463281e-15 -> 1.1750855152298039e-16 -1 -2.1665209362190277e-15
- joint l_ankle_pitch: axis -2.389602037081462e-16 1 1.4538275231733847e-16 -> -2.38960203708147e-16 1 1.4538275231733847e-16
- joint l_ankle_roll: axis 1 -4.05028482201375e-16 -1.2496691978128869e-15 -> 1 -4.050284822013754e-16 -1.2496691978128869e-15
- joint l_elbow: axis -8.847089727469744e-17 -0.9999999999999953 6.383782391594399e-15 -> -2.550043509679755e-16 -0.999999999999986 1.293409823688246e-14
- joint l_hip_pitch: axis -5.772831379991284e-17 -1 -1.3843833381666392e-17 -> -5.772831379991284e-17 -1 -1.384383338166718e-17
- joint l_hip_roll: axis 1 -6.123233995736708e-17 6.3201403498236e-16 -> 1 -6.123233995736708e-17 6.320140349823599e-16
- joint l_hip_yaw: axis -8.622588011769357e-16 1.5936665473077025e-16 1 -> -8.622588011769357e-16 1.5936665473077023e-16 1
- joint l_index_add: axis -3.232245792329867e-15 -0.9999999999999998 1.5397182495276352e-15 -> -3.3702260559116687e-15 -0.9999999999999993 1.0014973022447945e-15
- joint l_index_dist: axis -0.9999999999999997 1.2698175844150033e-15 1.3045120539345794e-15 -> -0.999999999999999 1.1587952819524896e-15 1.3045120539345763e-15
- joint l_index_prox: axis -0.9999999999999996 -2.0816681711721439e-16 3.99680288865056e-15 -> -0.9999999999999987 -3.1918911957972767e-16 4.024558464266183e-15
- joint l_knee: axis -2.608937546411318e-16 -1 5.166588955193111e-17 -> -2.60893754641131e-16 -1 5.166588955193113e-17
- joint l_middle_dist: axis -0.9999999999999998 -2.3467059288222403e-15 6.408211626924537e-16 -> -0.9999999999999993 -2.3467707837629264e-15 5.921449210147216e-16
- joint l_middle_prox: axis -0.9999999999999998 -1.0130785099575306e-15 -4.37150315993994e-16 -> -0.9999999999999993 -1.0685896612017132e-15 -4.78783679465276e-16
- joint l_pinkie_dist: axis -1.0000000000000002 -2.6194156222657784e-15 3.3662023329484224e-16 -> -1.0000000000000007 -2.6471672680994334e-15 3.0885679776748995e-16
- joint l_pinkie_prox: axis -1.0000000000000002 -1.1843525269243981e-15 5.273559366969494e-16 -> -1.0000000000000004 -1.1774136330204909e-15 4.996003610813204e-16
- joint l_ring_dist: axis -1.0000000000000002 -2.168404344970969e-17 1.2490009027033007e-15 -> -1.0000000000000007 -1.3270634591222456e-16 1.2351231148954863e-15
- joint l_ring_prox: axis -1.0000000000000002 -1.0100531863796072e-15 6.800116025829084e-16 -> -1.0000000000000004 -1.055155996755004e-15 6.522560269672795e-16
- joint l_shoulder_roll: axis 1 3.78169717762985e-16 2.7478019859473113e-15 -> 1 3.226585665316948e-16 2.775557561563002e-15
- joint l_shoulder_yaw: axis -3.00454106039183e-14 2.9143354396410367e-15 -0.9999999999999978 -> -6.00908212078363e-14 6.050715484207078e-15 -0.9999999999999933
- joint l_thumb_add: axis 3.3306690738754696e-16 -6.245004513516506e-16 -0.9999999999999998 -> 4.996003610813204e-16 -1.124100812432971e-15 -0.9999999999999993
- joint l_thumb_dist: axis -1.4016565559607482e-15 4.996003048844505e-16 -1 -> -1.901256909464961e-15 1.1102229532740747e-15 -1
- joint l_thumb_prox: axis 9.575673587391975e-16 -1.4988010832439613e-15 -1.0000000000000002 -> 4.163336342344337e-16 -9.992007221626409e-16 -1.0000000000000004
- joint l_wrist_pitch: axis -7.632783294297949e-17 -0.9999999999999999 -4.163336342344336e-16 -> -1.8735013540549497e-16 -0.9999999999999997 -1.0269562977782694e-15
- joint l_wrist_roll: axis -0.9999999999999999 4.805184028455756e-16 1.3877787807814474e-16 -> -0.9999999999999997 6.47051856539349e-16 7.632783294297998e-17
- joint l_wrist_yaw: axis -2.994132719535971e-14 2.9420910152566727e-15 -0.9999999999999982 -> -6.005612673831686e-14 5.828670879282063e-15 -0.9999999999999947
- joint r_ankle_pitch: axis -3.505264366441263e-17 1 -1.331317022347139e-16 -> -3.505264366441327e-17 1 -1.3313170223472496e-16
- joint r_ankle_roll: axis -1 -1.628246671334752e-16 2.560295622560413e-15 -> -1 -1.628246671334752e-16 2.5602956225604195e-15
- joint r_elbow: axis 2.4459601011270737e-16 -1.0000000000000027 1.2989609388114332e-14 -> 3.5561831257529417e-16 -1.000000000000008 2.5951463200613154e-14
- joint r_hip_pitch: axis -1.0880513989386065e-16 -1 1.384383338166008e-17 -> -1.0880513989386065e-16 -1 1.3843833381659292e-17
- joint r_hip_roll: axis -1 -3.3813287685016297e-16 -7.120227705451219e-17 -> -1 -3.3813287685016258e-16 -7.12022770545114e-17
- joint r_hip_yaw: axis -2.395305022015389e-20 1.474932849181089e-15 -1 -> -2.3953050200826797e-20 1.474932849181089e-15 -1
- joint r_index_add: axis -2.2710721778544278e-14 1.0000000000000058 -3.325533406549057e-15 -> -4.651242255183732e-14 1.0000000000000173 -6.08487548946725e-15
- joint r_index_dist: axis -1.0000000000000127 4.898859096158517e-14 -3.955169525227743e-16 -> -1.000000000000038 9.6672669869238e-14 -5.134781488895157e-16
- joint r_index_prox: axis -1.0000000000000127 4.871797409933279e-14 5.689893001203353e-16 -> -1.000000000000038 9.645756415821688e-14 3.8163916471455337e-16
- joint r_knee: axis 1.2193157766326317e-6 -0.9999999999992567 4.719551160658935e-15 -> 1.219315776632632e-6 -0.9999999999992569 4.719551160658948e-15
- joint r_middle_dist: axis -1.0000000000000127 4.8869412818017636e-14 7.711215903793126e-16 -> -1.000000000000038 9.694733146028018e-14 8.607486116259909e-16
- joint r_middle_prox: axis -1.0000000000000067 2.2546201017270685e-14 -2.45636844198318e-15 -> -1.00000000000002 4.66935518028684e-14 -2.470246229791037e-15
- joint r_pinkie_dist: axis -1.0000000000000142 4.6843605383539805e-14 1.91513471747844e-15 -> -1.0000000000000426 9.46109510180395e-14 2.164934898019344e-15
- joint r_pinkie_prox: axis -1.0000000000000073 2.687697787657948e-14 -2.761679773755077e-15 -> -1.0000000000000224 5.074677290602035e-14 -2.581268532253489e-15
- joint r_ring_dist: axis -1.0000000000000142 4.792260338559737e-14 -2.890049310977331e-15 -> -1.0000000000000426 9.566219344448145e-14 -2.647188024340446e-15
- joint r_ring_prox: axis -1.0000000000000073 2.7031320490650422e-14 -2.5396351688300456e-15 -> -1.0000000000000222 5.091846275485106e-14 -2.345346139520643e-15
- joint r_shoulder_roll: axis -1.0000000000000009 8.205242041369425e-16 1.734723475977312e-16 -> -1.0000000000000027 1.153591111524405e-15 1.9428902930949706e-16
- joint r_shoulder_yaw: axis -4.579669976578765e-16 5.551115123125817e-17 1 -> -4.371503159461546e-16 8.32667268468839e-17 1
- joint r_thumb_add: axis 1.304512053934559e-15 4.801714581503802e-15 1.0000000000000062 -> 3.3584246494910985e-15 1.0560996521746802e-14 1.0000000000000187
- joint r_thumb_dist: axis -5.290212712338784e-14 -2.997602166487913e-14 -1.0000000000000502 -> -1.5804024755539139e-13 -8.88733531212472e-14 -1.0000000000001505
- joint r_thumb_prox: axis -3.549938121238938e-14 -1.840194663316197e-14 -1.0000000000000255 -> -7.101264021258658e-14 -3.7719827261639693e-14 -1.0000000000000764
- joint r_wrist_pitch: axis 5.100087019371814e-16 -1 -5.273559366969494e-16 -> 4.544975507059239e-16 -1 -1.1379786002407858e-15
- joint r_wrist_roll: axis 1.0000000000000004 -1.8735013540549512e-16 7.632783294297946e-17 -> 1.0000000000000013 -2.42861286636753e-16 4.857225732735043e-17
- joint r_wrist_yaw: axis 5.7037707890117685e-15 -1.2517764602648659e-14 1.0000000000000022 -> 1.1289580381657174e-14 -2.514655150775995e-14 1.0000000000000067
- joint torso_pitch: axis 1.9259299443837326e-34 1 0 -> 3.851859888763962e-34 1 0
