Commit message: Update ergoCubSN001 with neck mk3 (#370)

File: urdf/ergoCub/robots/ergoCubGazeboSN000/model.urdf (robot description, URDF)
Before this commit: robot ergoCub, 204 links, 203 joints
Links:
- link chest: geometry collision mesh filename=package://ergoCub/meshes/simmechanics/sim_ecub_1-1_chest.stl scale=0.001 0.001 0.001; visual mesh filename=package://ergoCub/meshes/simmechanics/sim_ecub_1-1_chest.stl scale=0.001 0.001 0.001
- link head: geometry collision mesh filename=package://ergoCub/meshes/simmechanics/sim_ecub_1-1_head.stl scale=0.001 0.001 0.001; visual mesh filename=package://ergoCub/meshes/simmechanics/sim_ecub_1-1_head.stl scale=0.001 0.001 0.001

File: urdf/ergoCub/robots/ergoCubGazeboSN000_minContacts/model.urdf (robot description, URDF)
Before this commit: robot ergoCub, 204 links, 203 joints
Links:
- link chest: geometry visual mesh filename=package://ergoCub/meshes/simmechanics/sim_ecub_1-1_chest.stl scale=0.001 0.001 0.001
- link head: geometry visual mesh filename=package://ergoCub/meshes/simmechanics/sim_ecub_1-1_head.stl scale=0.001 0.001 0.001

File: urdf/ergoCub/robots/ergoCubGazeboSN001/model.urdf (robot description, URDF)
Before this commit: robot ergoCub, 204 links, 203 joints
Links:
- added link neck_1, mass 0.25627387976979793; collision mesh filename=package://ergoCub/meshes/simmechanics/sim_ecub_1-3_head_nec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 scale=0.001 0.001 0.001; visual mesh filename=package://ergoCub/meshes/simmechanics/sim_ecub_1-3_head_nec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 scale=0.001 0.001 0.001
- link chest: mass 8.065471632648594 -> 8.302489936617166; geometry collision mesh filename=package://ergoCub/meshes/simmechanics/sim_ecub_1-1_chest_wo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 scale=0.001 0.001 0.001; visual mesh filename=package://ergoCub/meshes/simmechanics/sim_ecub_1-1_chest_wo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 scale=0.001 0.001 0.001
- link head: mass 1.972127893184972 -> 1.6902682; geometry collision mesh filename=package://ergoCub/meshes/simmechanics/sim_ecub_1-1_head.stl scale=0.001 0.001 0.001; visual mesh filename=package://ergoCub/meshes/simmechanics/sim_ecub_1-1_head.stl scale=0.001 0.001 0.001
- link neck_2: mass 0.12100314943032965 -> 0.2945770397905417; geometry collision mesh filename=package://ergoCub/meshes/simmechanics/sim_ecub_1-3_head_nec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 scale=0.001 0.001 0.001; visual mesh filename=package://ergoCub/meshes/simmechanics/sim_ecub_1-3_head_nec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 scale=0.001 0.001 0.001
- link neck_3: mass 0.17811376821431446 -> 0.26196252682452986; geometry collision mesh filename=package://ergoCub/meshes/simmechanics/sim_ecub_1-3_head_nec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 scale=0.001 0.001 0.001; visual mesh filename=package://ergoCub/meshes/simmechanics/sim_ecub_1-3_head_nec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 scale=0.001 0.001 0.001
Joints:
- added joint neck_fixed_joint: type fixed, parent chest, child neck_1, origin xyz=-0.0037884876520280393 2.689105939166276e-16 0.18030000000000007 rpy=-2.2171138790649083e-15 -1.991357518387602e-15 -2.8831104173325634e-15
- joint camera_tilt: axis -3.1332662159460226e-17 -1 -1.3036401662462866e-15 -> -1.998015835203486e-13 -1 -8.597927048660853e-14; origin xyz=0.06250999999999993 -3.0000000001105853e-5 0.07639250000000064 rpy=9.166950960511526e-15 2.595819949100105e-4 1.9343583275079285e-15 -> xyz=0.06250999999999991 -2.999999997621366e-5 0.07639249999999997 rpy=-7.545682259870277e-14 2.5958199361694967e-4 2.017046159162252e-13
- joint l_arm_ft_sensor: origin xyz=-0.004349999999999986 -2.7755575615628914e-17 -0.05430000000000004 rpy=2.2204460492503136e-16 6.938893903907228e-18 1.4988010832439621e-15 -> xyz=-0.004350000000000007 2.7755575615628914e-17 -0.05430000000000004 rpy=2.498001805406603e-16 6.938893903907228e-18 1.4988010832439623e-15
- joint l_index_add: axis 1.1895336853461886e-15 0.9999999999999999 -1.9812040713213337e-15 -> 1.1895336853461886e-15 1 -2.0089596469369626e-15; origin xyz=0.022500000000000023 -0.0015000000000006952 -0.0685999999999996 rpy=-8.416895217637947e-16 -0.29670597224465534 5.804755322508926e-17 -> xyz=0.02250000000000001 -0.0015000000000006397 -0.0685999999999996 rpy=-8.707132983763394e-16 -0.29670597224465534 5.804755322508926e-17
- joint l_index_dist: axis -1 -2.359224176539984e-16 4.163337069211178e-17 -> -1 -2.9143356888525625e-16 9.714452192336961e-17; origin xyz=-1.3877787807814457e-17 -0.001500000000000029 -0.03999999999999987 rpy=-7.482326172536535e-8 1.8041124150158794e-16 -6.106226635438361e-16 -> xyz=-2.7755575615628914e-17 -0.0015000000000000013 -0.03999999999999987 rpy=-7.482326172536535e-8 1.8041124150158794e-16 -5.551115123125783e-16
- joint l_index_prox: axis -1 8.326672684688522e-17 7.023654435833748e-10 -> -1 8.326672684688543e-17 7.023654366444809e-10; origin xyz=0.00919253334679343 0 -0.030713451309624218 rpy=-3.0531133177191815e-16 -7.023611484080483e-10 -7.771561172376096e-16 -> xyz=0.009192533346793444 0 -0.030713451309624218 rpy=-2.7755575615628923e-16 -7.02361099835791e-10 -8.326672684688674e-16
- joint l_shoulder_pitch: axis -3.452099717193846e-16 1.0000000000000002 3.0531133177191805e-16 -> -4.5102810375396984e-17 1 -8.326672684688674e-17; origin xyz=-0.013518676842610159 0.06704761117227499 0.12351981080941767 rpy=0.2536123238732541 -0.05203160550449479 -0.27527873241387235 -> xyz=-0.013518676842610003 0.06704761117227499 0.1235198108094176 rpy=0.25361232387325433 -0.05203160550449447 -0.2752787324138737
- joint l_shoulder_roll: axis 1 4.891920202255013e-16 3.3029134982598896e-15 -> 1 2.671474153004699e-16 2.768618667659033e-15; origin xyz=0.005000000000000011 0.09329999999999987 -3.0531133177191805e-16 rpy=2.6895152771544417e-14 1.790234627208065e-15 -2.3314683517128287e-15 -> xyz=0.005000000000000025 0.09330000000000005 -1.1102230246251565e-16 rpy=2.6839641620313153e-14 1.2559397966072083e-15 -2.1094237467877974e-15
- joint l_shoulder_yaw: axis -3.0080105073437835e-14 3.191891195797326e-15 -0.9999999999999977 -> -2.988581604412843e-14 3.3029134982598415e-15 -0.9999999999999976; origin xyz=4.163336342344337e-17 -5.551115123125783e-17 -0.022499999999999937 rpy=-3.3029134982598486e-15 -3.002459392220658e-14 6.383782391594671e-15 -> xyz=-1.3877787807814457e-17 -2.7755575615628914e-16 -0.022500000000000075 rpy=-3.4139358007223646e-15 -2.9830304892897175e-14 5.884182030513349e-15
- joint neck_pitch: axis 2.6472211157644926e-18 -1 -7.807858529815144e-16 -> -6.696259655795151e-17 -1 -2.736197492574649e-16; origin xyz=0.004861512347971912 4.1253975310307907e-16 0.22529999999999994 rpy=-1.541978321110266e-15 -2.0480667158215426e-15 -1.389802281096855e-15 -> xyz=0.008650000000000036 3.477503656126425e-17 0.04500000000000004 rpy=-2.736197492574658e-16 7.317379024648131e-17 6.696259655795151e-17; parent chest -> neck_1
- joint neck_roll: axis 1 -1.6820355477448088e-15 -3.806893332301044e-15 -> 1 2.30576840860686e-16 -7.196923107658096e-17; limit lower=-0.3490658503988659 upper=0.3490658503988659 effort=1e+9 velocity=1e+9 -> lower=-0.5235987755982988 upper=0.5235987755982988 effort=1e+9 velocity=1e+9; origin xyz=8.673617379884035e-19 6.416192023745373e-17 0.009499999999999786 rpy=-1.7364294099408703e-15 -2.980403162017727e-16 1.580860396783509e-15 -> xyz=-3.5561831257524545e-17 7.375606977361926e-16 0.010999999999997845 rpy=8.452269018635315e-14 7.050925500045285e-14 1.2263451870709675e-14
- joint neck_yaw: axis 3.1628618281392715e-15 1.6479574685948862e-15 0.9999999999999998 -> 1.386477883657293e-15 2.1582026845669262e-16 0.9999999999999999; origin xyz=-1.43982048506075e-16 -4.1419339784385294e-17 0.06914999999999999 rpy=1.2720090288173385e-15 -3.1687776687987536e-15 3.715432083235576e-16 -> xyz=-1.734723475976807e-18 1.0057301276633031e-23 0.06914999999999993 rpy=2.1582026845669264e-16 -1.386477883657293e-15 -1.9981249037222812e-13
- joint r_arm_ft_sensor: origin xyz=-0.006850000000000004 -5.551115123125783e-17 -0.054300000000000015 rpy=-2.220446049250312e-16 -2.3592239273284576e-16 1.6098233857064762e-15 -> xyz=-0.006849999999999993 0 -0.05429999999999999 rpy=-1.6653345369377346e-16 -2.2898349882893854e-16 1.7763568394002497e-15
- joint r_shoulder_pitch: axis -2.445960101127298e-16 1 3.552713678800501e-15 -> -2.1337098754514727e-16 1.0000000000000002 3.6637359812630166e-15; origin xyz=-0.013518676842610352 -0.06704761117227452 0.12351981080941783 rpy=-0.25361232387326116 -0.05203160550449495 0.2752787324138702 -> xyz=-0.013518676842610456 -0.06704761117227441 0.12351981080941779 rpy=-0.2536123238732615 -0.052031605504494885 0.2752787324138686
- joint r_shoulder_roll: axis -1.0000000000000007 8.760353553682006e-16 -4.510281037539194e-16 -> -1.0000000000000007 1.042568809061973e-15 -6.869504964867667e-16; origin xyz=0.007499999999999977 -0.09330000000000004 -3.885780586188048e-16 rpy=-9.325873406851307e-15 9.520162436160717e-15 -4.718447854656912e-15 -> xyz=0.007499999999999915 -0.09329999999999992 -4.718447854656915e-16 rpy=-9.270362255620051e-15 9.783840404509192e-15 -4.6074255521943965e-15
- joint r_shoulder_yaw: axis 2.567390744445681e-16 2.775557561562927e-17 1.0000000000000004 -> 5.551115123125789e-16 2.775557561562895e-16 1.0000000000000002; origin xyz=-7.979727989493313e-17 5.551115123125783e-17 -0.02249999999999998 rpy=-5.55111512312578e-17 -3.0531133177191805e-16 7.660538869913577e-15 -> xyz=-2.7755575615628914e-17 -1.3877787807814457e-16 -0.02249999999999991 rpy=1.9428902930940235e-16 -6.036837696399289e-16 7.494005416219803e-15
- joint torso_pitch: axis 1.058791184074231e-22 1 4.336808689942018e-19 -> 7.006492321624082e-46 1 0; origin xyz=-7.30886630439206e-17 -4.930380657631324e-32 0.11800000000000001 rpy=3.9719461100401744e-15 2.710505431213761e-20 1.0587911275090697e-22 -> xyz=-7.308866350978873e-17 -9.860761315262648e-32 0.11800000000000001 rpy=3.972379790909169e-15 7.822717473246975e-47 -5.656623812198895e-30
- joint torso_roll: axis -1 0 1.4239886692466155e-15 -> -1 -3.7495681564941394e-46 1.4239886692466155e-15; origin xyz=-2.23890229767886e-18 -5.551115123142428e-20 0.060500000000000095 rpy=0 -2.2470258116354473e-44 5.656623812198896e-30 -> xyz=-2.29578282319141e-18 1.637578961322135e-18 0.06050000000000004 rpy=1.3877787807814457e-17 -2.239175669138015e-44 5.6368619996063595e-30
- joint torso_yaw: axis 2.084864385226231e-15 -2.114127025714114e-15 -1 -> 2.084865167540359e-15 -2.1136160009445084e-15 -1; origin xyz=7.32502235717738e-17 2.561326957877574e-16 0.0644699999999999 rpy=-3.971868545919581e-15 -4.385099568445115e-23 -3.1763738272196853e-22 -> xyz=7.323422676005885e-17 2.5446174810332376e-16 0.06446999999999997 rpy=-3.97237957068919e-15 7.384631424546912e-22 1.6549261963221894e-15

File: urdf/ergoCub/robots/ergoCubGazeboSN001_minContacts/model.urdf (robot description, URDF)
Before this commit: robot ergoCub, 204 links, 203 joints
Links:
- added link neck_1, mass 0.25627387976979793; visual mesh filename=package://ergoCub/meshes/simmechanics/sim_ecub_1-3_head_nec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 scale=0.001 0.001 0.001
- link chest: mass 8.065471632648594 -> 8.302489936617166; geometry visual mesh filename=package://ergoCub/meshes/simmechanics/sim_ecub_1-1_chest_wo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 scale=0.001 0.001 0.001
- link head: mass 1.972127893184972 -> 1.6902682; geometry visual mesh filename=package://ergoCub/meshes/simmechanics/sim_ecub_1-1_head.stl scale=0.001 0.001 0.001
- link neck_2: mass 0.12100314943032965 -> 0.2945770397905417; geometry visual mesh filename=package://ergoCub/meshes/simmechanics/sim_ecub_1-3_head_nec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 scale=0.001 0.001 0.001
- link neck_3: mass 0.17811376821431446 -> 0.26196252682452986; geometry visual mesh filename=package://ergoCub/meshes/simmechanics/sim_ecub_1-3_head_nec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 scale=0.001 0.001 0.001
Joints:
- added joint neck_fixed_joint: type fixed, parent chest, child neck_1, origin xyz=-0.0037884876520280393 2.689105939166276e-16 0.18030000000000007 rpy=-2.2171138790649083e-15 -1.991357518387602e-15 -2.8831104173325634e-15
- joint camera_tilt: axis -3.1332662159460226e-17 -1 -1.3036401662462866e-15 -> -1.998015835203486e-13 -1 -8.597927048660853e-14; origin xyz=0.06250999999999993 -3.0000000001105853e-5 0.07639250000000064 rpy=9.166950960511526e-15 2.595819949100105e-4 1.9343583275079285e-15 -> xyz=0.06250999999999991 -2.999999997621366e-5 0.07639249999999997 rpy=-7.545682259870277e-14 2.5958199361694967e-4 2.017046159162252e-13
- joint l_arm_ft_sensor: origin xyz=-0.004349999999999986 -2.7755575615628914e-17 -0.05430000000000004 rpy=2.2204460492503136e-16 6.938893903907228e-18 1.4988010832439621e-15 -> xyz=-0.004350000000000007 2.7755575615628914e-17 -0.05430000000000004 rpy=2.498001805406603e-16 6.938893903907228e-18 1.4988010832439623e-15
- joint l_index_add: axis 1.1895336853461886e-15 0.9999999999999999 -1.9812040713213337e-15 -> 1.1895336853461886e-15 1 -2.0089596469369626e-15; origin xyz=0.022500000000000023 -0.0015000000000006952 -0.0685999999999996 rpy=-8.416895217637947e-16 -0.29670597224465534 5.804755322508926e-17 -> xyz=0.02250000000000001 -0.0015000000000006397 -0.0685999999999996 rpy=-8.707132983763394e-16 -0.29670597224465534 5.804755322508926e-17
- joint l_index_dist: axis -1 -2.359224176539984e-16 4.163337069211178e-17 -> -1 -2.9143356888525625e-16 9.714452192336961e-17; origin xyz=-1.3877787807814457e-17 -0.001500000000000029 -0.03999999999999987 rpy=-7.482326172536535e-8 1.8041124150158794e-16 -6.106226635438361e-16 -> xyz=-2.7755575615628914e-17 -0.0015000000000000013 -0.03999999999999987 rpy=-7.482326172536535e-8 1.8041124150158794e-16 -5.551115123125783e-16
- joint l_index_prox: axis -1 8.326672684688522e-17 7.023654435833748e-10 -> -1 8.326672684688543e-17 7.023654366444809e-10; origin xyz=0.00919253334679343 0 -0.030713451309624218 rpy=-3.0531133177191815e-16 -7.023611484080483e-10 -7.771561172376096e-16 -> xyz=0.009192533346793444 0 -0.030713451309624218 rpy=-2.7755575615628923e-16 -7.02361099835791e-10 -8.326672684688674e-16
- joint l_shoulder_pitch: axis -3.452099717193846e-16 1.0000000000000002 3.0531133177191805e-16 -> -4.5102810375396984e-17 1 -8.326672684688674e-17; origin xyz=-0.013518676842610159 0.06704761117227499 0.12351981080941767 rpy=0.2536123238732541 -0.05203160550449479 -0.27527873241387235 -> xyz=-0.013518676842610003 0.06704761117227499 0.1235198108094176 rpy=0.25361232387325433 -0.05203160550449447 -0.2752787324138737
- joint l_shoulder_roll: axis 1 4.891920202255013e-16 3.3029134982598896e-15 -> 1 2.671474153004699e-16 2.768618667659033e-15; origin xyz=0.005000000000000011 0.09329999999999987 -3.0531133177191805e-16 rpy=2.6895152771544417e-14 1.790234627208065e-15 -2.3314683517128287e-15 -> xyz=0.005000000000000025 0.09330000000000005 -1.1102230246251565e-16 rpy=2.6839641620313153e-14 1.2559397966072083e-15 -2.1094237467877974e-15
- joint l_shoulder_yaw: axis -3.0080105073437835e-14 3.191891195797326e-15 -0.9999999999999977 -> -2.988581604412843e-14 3.3029134982598415e-15 -0.9999999999999976; origin xyz=4.163336342344337e-17 -5.551115123125783e-17 -0.022499999999999937 rpy=-3.3029134982598486e-15 -3.002459392220658e-14 6.383782391594671e-15 -> xyz=-1.3877787807814457e-17 -2.7755575615628914e-16 -0.022500000000000075 rpy=-3.4139358007223646e-15 -2.9830304892897175e-14 5.884182030513349e-15
- joint neck_pitch: axis 2.6472211157644926e-18 -1 -7.807858529815144e-16 -> -6.696259655795151e-17 -1 -2.736197492574649e-16; origin xyz=0.004861512347971912 4.1253975310307907e-16 0.22529999999999994 rpy=-1.541978321110266e-15 -2.0480667158215426e-15 -1.389802281096855e-15 -> xyz=0.008650000000000036 3.477503656126425e-17 0.04500000000000004 rpy=-2.736197492574658e-16 7.317379024648131e-17 6.696259655795151e-17; parent chest -> neck_1
- joint neck_roll: axis 1 -1.6820355477448088e-15 -3.806893332301044e-15 -> 1 2.30576840860686e-16 -7.196923107658096e-17; limit lower=-0.3490658503988659 upper=0.3490658503988659 effort=1e+9 velocity=1e+9 -> lower=-0.5235987755982988 upper=0.5235987755982988 effort=1e+9 velocity=1e+9; origin xyz=8.673617379884035e-19 6.416192023745373e-17 0.009499999999999786 rpy=-1.7364294099408703e-15 -2.980403162017727e-16 1.580860396783509e-15 -> xyz=-3.5561831257524545e-17 7.375606977361926e-16 0.010999999999997845 rpy=8.452269018635315e-14 7.050925500045285e-14 1.2263451870709675e-14
- joint neck_yaw: axis 3.1628618281392715e-15 1.6479574685948862e-15 0.9999999999999998 -> 1.386477883657293e-15 2.1582026845669262e-16 0.9999999999999999; origin xyz=-1.43982048506075e-16 -4.1419339784385294e-17 0.06914999999999999 rpy=1.2720090288173385e-15 -3.1687776687987536e-15 3.715432083235576e-16 -> xyz=-1.734723475976807e-18 1.0057301276633031e-23 0.06914999999999993 rpy=2.1582026845669264e-16 -1.386477883657293e-15 -1.9981249037222812e-13
- joint r_arm_ft_sensor: origin xyz=-0.006850000000000004 -5.551115123125783e-17 -0.054300000000000015 rpy=-2.220446049250312e-16 -2.3592239273284576e-16 1.6098233857064762e-15 -> xyz=-0.006849999999999993 0 -0.05429999999999999 rpy=-1.6653345369377346e-16 -2.2898349882893854e-16 1.7763568394002497e-15
- joint r_shoulder_pitch: axis -2.445960101127298e-16 1 3.552713678800501e-15 -> -2.1337098754514727e-16 1.0000000000000002 3.6637359812630166e-15; origin xyz=-0.013518676842610352 -0.06704761117227452 0.12351981080941783 rpy=-0.25361232387326116 -0.05203160550449495 0.2752787324138702 -> xyz=-0.013518676842610456 -0.06704761117227441 0.12351981080941779 rpy=-0.2536123238732615 -0.052031605504494885 0.2752787324138686
- joint r_shoulder_roll: axis -1.0000000000000007 8.760353553682006e-16 -4.510281037539194e-16 -> -1.0000000000000007 1.042568809061973e-15 -6.869504964867667e-16; origin xyz=0.007499999999999977 -0.09330000000000004 -3.885780586188048e-16 rpy=-9.325873406851307e-15 9.520162436160717e-15 -4.718447854656912e-15 -> xyz=0.007499999999999915 -0.09329999999999992 -4.718447854656915e-16 rpy=-9.270362255620051e-15 9.783840404509192e-15 -4.6074255521943965e-15
- joint r_shoulder_yaw: axis 2.567390744445681e-16 2.775557561562927e-17 1.0000000000000004 -> 5.551115123125789e-16 2.775557561562895e-16 1.0000000000000002; origin xyz=-7.979727989493313e-17 5.551115123125783e-17 -0.02249999999999998 rpy=-5.55111512312578e-17 -3.0531133177191805e-16 7.660538869913577e-15 -> xyz=-2.7755575615628914e-17 -1.3877787807814457e-16 -0.02249999999999991 rpy=1.9428902930940235e-16 -6.036837696399289e-16 7.494005416219803e-15
- joint torso_pitch: axis 1.058791184074231e-22 1 4.336808689942018e-19 -> 7.006492321624082e-46 1 0; origin xyz=-7.30886630439206e-17 -4.930380657631324e-32 0.11800000000000001 rpy=3.9719461100401744e-15 2.710505431213761e-20 1.0587911275090697e-22 -> xyz=-7.308866350978873e-17 -9.860761315262648e-32 0.11800000000000001 rpy=3.972379790909169e-15 7.822717473246975e-47 -5.656623812198895e-30
- joint torso_roll: axis -1 0 1.4239886692466155e-15 -> -1 -3.7495681564941394e-46 1.4239886692466155e-15; origin xyz=-2.23890229767886e-18 -5.551115123142428e-20 0.060500000000000095 rpy=0 -2.2470258116354473e-44 5.656623812198896e-30 -> xyz=-2.29578282319141e-18 1.637578961322135e-18 0.06050000000000004 rpy=1.3877787807814457e-17 -2.239175669138015e-44 5.6368619996063595e-30
- joint torso_yaw: axis 2.084864385226231e-15 -2.114127025714114e-15 -1 -> 2.084865167540359e-15 -2.1136160009445084e-15 -1; origin xyz=7.32502235717738e-17 2.561326957877574e-16 0.0644699999999999 rpy=-3.971868545919581e-15 -4.385099568445115e-23 -3.1763738272196853e-22 -> xyz=7.323422676005885e-17 2.5446174810332376e-16 0.06446999999999997 rpy=-3.97237957068919e-15 7.384631424546912e-22 1.6549261963221894e-15

File: urdf/ergoCub/robots/ergoCubGazeboSN003/model.urdf (robot description, URDF)
Before this commit: robot ergoCub, 205 links, 204 joints
Joints:
- joint neck_roll: limit lower=-0.3490658503988659 upper=0.3490658503988659 effort=1e+9 velocity=1e+9 -> lower=-0.5235987755982988 upper=0.5235987755982988 effort=1e+9 velocity=1e+9

File: urdf/ergoCub/robots/ergoCubGazeboSN003_minContacts/model.urdf (robot description, URDF)
Before this commit: robot ergoCub, 205 links, 204 joints
Joints:
- joint neck_roll: limit lower=-0.3490658503988659 upper=0.3490658503988659 effort=1e+9 velocity=1e+9 -> lower=-0.5235987755982988 upper=0.5235987755982988 effort=1e+9 velocity=1e+9

File: urdf/ergoCub/robots/ergoCubSN000/model.urdf (robot description, URDF)
Before this commit: robot ergoCub, 204 links, 203 joints
Links:
- link chest: geometry collision mesh filename=package://ergoCub/meshes/simmechanics/sim_ecub_1-1_chest.stl scale=0.001 0.001 0.001; visual mesh filename=package://ergoCub/meshes/simmechanics/sim_ecub_1-1_chest.stl scale=0.001 0.001 0.001
- link head: geometry collision mesh filename=package://ergoCub/meshes/simmechanics/sim_ecub_1-1_head.stl scale=0.001 0.001 0.001; visual mesh filename=package://ergoCub/meshes/simmechanics/sim_ecub_1-1_head.stl scale=0.001 0.001 0.001
