Commit message: Automatic update of urdf triggered by GitHub Action
ergocub-software = c4fbfdd12bf22a6ace0f4a9719dcd183f753bbcb
cad-libraries    = https://github.com/mesh-iit/cad-libraries/commit/39d958532d47ec17332b42330f3711c516e857bc
cad-mechanics    = https://github.com/mesh-iit/cad-mechanics/commit/f5367584f40cdfd19934d7a8fedfc16edcca747b
creo2urdf        = https://github.com/mesh-iit/creo2urdf/releases/tag/v0.5.18

File: urdf/ergoCub/robots/ergoCubGazeboSN000/model.urdf (robot description, URDF)
Before this commit: robot ergoCub, 204 links, 203 joints
Links:
- link realsense: mass 0.0973042045264468 -> 0.08233251527028056
Joints:
- joint camera_tilt: axis 1.9074075506529947e-16 -1 -1.4146048262463281e-15 -> -7.529259780358045e-16 -1 -5.660091301660127e-16; origin xyz=0.06251 -3.0000000001127547e-5 0.0763925000000007 rpy=9.055928654249867e-15 2.5958199361703294e-4 1.7122849027886369e-15 -> xyz=0.06250999999999989 -3.0000000001138484e-5 0.07639250000000042 rpy=9.528820759122059e-15 2.595819932592144e-4 2.6559516676797224e-15
- joint l_index_dist: axis -0.9999999999999997 1.2698175844150033e-15 1.3045120539345794e-15 -> -0.9999999999999999 1.3253287356462613e-15 1.2351231148955076e-15; origin xyz=4.163336342344337e-17 -0.0015000000000000013 -0.030000000000000082 rpy=-1.6320278461989814e-14 -1.1102230246251565e-16 1.110223024625157e-16 -> xyz=2.7755575615628914e-17 -0.0015000000000000568 -0.02999999999999997 rpy=-1.6320278461989807e-14 -5.551115123125783e-17 5.551115123125784e-17
- joint l_index_prox: axis -0.9999999999999996 -2.0816681711721439e-16 3.99680288865056e-15 -> -0.9999999999999998 -2.0816681711721453e-16 3.996802888650561e-15; origin xyz=0.009192533317427712 -2.7755575615628914e-17 -0.030713451316238316 rpy=6.383782391594655e-16 -1.942890293094024e-16 1.110223024625157e-16 -> xyz=0.00919253331742774 0 -0.030713451316238427 rpy=6.106226635438364e-16 -2.636779683484747e-16 5.551115123125784e-17
- joint neck_yaw: axis 1.4082090529075477e-15 5.709519748275242e-16 0.9999999999999998 -> 1.6591628191298083e-15 5.987076998014226e-16 0.9999999999999998; origin xyz=-1.3010426069826053e-17 3.765597982987134e-17 0.0691500000000001 rpy=1.9500353504997633e-16 -1.4141248935670295e-15 3.767470613092508e-16 -> xyz=-4.0766001685454967e-17 3.151498988337666e-17 0.0691500000000001 rpy=2.2275926002387476e-16 -1.6650786597892902e-15 3.2676263100504264e-16
- joint realsense_depth_frame_fixed_joint: origin xyz=0.007515481871156526 0.010000000000000002 1.7352099479506222e-8 rpy=-1.5707963267948966 3.7596758519972983e-16 -1.5707963267948966 -> xyz=0.007415481871156544 0.047499999999999994 1.735209986808428e-8 rpy=-1.5707963267948966 1.439727114483606e-19 -1.570796326794897
- joint realsense_imu_0_fixed_joint: origin xyz=0.007515481871156526 0.010000000000000002 1.7352099479506222e-8 rpy=-1.5707963267948966 3.7596758519972983e-16 -1.5707963267948966 -> xyz=0.007415481871156544 0.047499999999999994 1.735209986808428e-8 rpy=-1.5707963267948966 1.439727114483606e-19 -1.570796326794897
- joint realsense_rgb_frame_fixed_joint: origin xyz=0.007515481871156526 -0.011499999999999996 1.7352099701550827e-8 rpy=-1.5707963267948966 3.7596758519972983e-16 -1.5707963267948966 -> xyz=0.007415481871156544 -0.011499999999999993 1.735209981257313e-8 rpy=-1.5707963267948966 1.439727114483606e-19 -1.570796326794897

File: urdf/ergoCub/robots/ergoCubGazeboSN000_minContacts/model.urdf (robot description, URDF)
Before this commit: robot ergoCub, 204 links, 203 joints
Links:
- link realsense: mass 0.0973042045264468 -> 0.08233251527028056
Joints:
- joint camera_tilt: axis 1.9074075506529947e-16 -1 -1.4146048262463281e-15 -> -7.529259780358045e-16 -1 -5.660091301660127e-16; origin xyz=0.06251 -3.0000000001127547e-5 0.0763925000000007 rpy=9.055928654249867e-15 2.5958199361703294e-4 1.7122849027886369e-15 -> xyz=0.06250999999999989 -3.0000000001138484e-5 0.07639250000000042 rpy=9.528820759122059e-15 2.595819932592144e-4 2.6559516676797224e-15
- joint l_index_dist: axis -0.9999999999999997 1.2698175844150033e-15 1.3045120539345794e-15 -> -0.9999999999999999 1.3253287356462613e-15 1.2351231148955076e-15; origin xyz=4.163336342344337e-17 -0.0015000000000000013 -0.030000000000000082 rpy=-1.6320278461989814e-14 -1.1102230246251565e-16 1.110223024625157e-16 -> xyz=2.7755575615628914e-17 -0.0015000000000000568 -0.02999999999999997 rpy=-1.6320278461989807e-14 -5.551115123125783e-17 5.551115123125784e-17
- joint l_index_prox: axis -0.9999999999999996 -2.0816681711721439e-16 3.99680288865056e-15 -> -0.9999999999999998 -2.0816681711721453e-16 3.996802888650561e-15; origin xyz=0.009192533317427712 -2.7755575615628914e-17 -0.030713451316238316 rpy=6.383782391594655e-16 -1.942890293094024e-16 1.110223024625157e-16 -> xyz=0.00919253331742774 0 -0.030713451316238427 rpy=6.106226635438364e-16 -2.636779683484747e-16 5.551115123125784e-17
- joint neck_yaw: axis 1.4082090529075477e-15 5.709519748275242e-16 0.9999999999999998 -> 1.6591628191298083e-15 5.987076998014226e-16 0.9999999999999998; origin xyz=-1.3010426069826053e-17 3.765597982987134e-17 0.0691500000000001 rpy=1.9500353504997633e-16 -1.4141248935670295e-15 3.767470613092508e-16 -> xyz=-4.0766001685454967e-17 3.151498988337666e-17 0.0691500000000001 rpy=2.2275926002387476e-16 -1.6650786597892902e-15 3.2676263100504264e-16
- joint realsense_depth_frame_fixed_joint: origin xyz=0.007515481871156526 0.010000000000000002 1.7352099479506222e-8 rpy=-1.5707963267948966 3.7596758519972983e-16 -1.5707963267948966 -> xyz=0.007415481871156544 0.047499999999999994 1.735209986808428e-8 rpy=-1.5707963267948966 1.439727114483606e-19 -1.570796326794897
- joint realsense_imu_0_fixed_joint: origin xyz=0.007515481871156526 0.010000000000000002 1.7352099479506222e-8 rpy=-1.5707963267948966 3.7596758519972983e-16 -1.5707963267948966 -> xyz=0.007415481871156544 0.047499999999999994 1.735209986808428e-8 rpy=-1.5707963267948966 1.439727114483606e-19 -1.570796326794897
- joint realsense_rgb_frame_fixed_joint: origin xyz=0.007515481871156526 -0.011499999999999996 1.7352099701550827e-8 rpy=-1.5707963267948966 3.7596758519972983e-16 -1.5707963267948966 -> xyz=0.007415481871156544 -0.011499999999999993 1.735209981257313e-8 rpy=-1.5707963267948966 1.439727114483606e-19 -1.570796326794897

File: urdf/ergoCub/robots/ergoCubGazeboSN001/model.urdf (robot description, URDF)
Before this commit: robot ergoCub, 205 links, 204 joints
Links:
- link realsense: mass 0.0973042045264468 -> 0.08233251527028056
Joints:
- joint camera_tilt: axis -1.998015835203486e-13 -1 -8.597927048660853e-14 -> -7.529259780358163e-16 -1 -5.660091301660221e-16; origin xyz=0.06250999999999991 -2.999999997621366e-5 0.07639249999999997 rpy=-7.545682259870277e-14 2.5958199361694967e-4 2.017046159162252e-13 -> xyz=0.06250999999999987 -3.000000000113848e-5 0.07639250000000047 rpy=9.528820759122057e-15 2.5958199325913113e-4 2.6559516676797335e-15
- joint l_index_dist: axis -1 -2.9143356888525625e-16 9.714452192336961e-17 -> -1.0000000000000002 -2.359224176539984e-16 1.457167792507203e-16; origin xyz=-2.7755575615628914e-17 -0.0015000000000000013 -0.03999999999999987 rpy=-7.482326172536535e-8 1.8041124150158794e-16 -5.551115123125783e-16 -> xyz=-2.7755575615628914e-17 -0.0014999999999999736 -0.039999999999999925 rpy=-7.482326169760975e-8 1.734723475976807e-16 -5.551115123125782e-16
- joint neck_roll: axis 1 2.30576840860686e-16 -7.196923107658096e-17 -> 1 2.3057684086068286e-16 -7.196923107658096e-17
- joint neck_yaw: axis 1.386477883657293e-15 2.1582026845669262e-16 0.9999999999999999 -> 1.3309667326328268e-15 1.603091172356458e-16 0.9999999999999999; origin xyz=-1.734723475976807e-18 1.0057301276633031e-23 0.06914999999999993 rpy=2.1582026845669264e-16 -1.386477883657293e-15 -1.9981249037222812e-13 -> xyz=-5.0306980803327406e-17 2.0696535769897827e-17 0.06914999999999971 rpy=1.6030911723564583e-16 -1.3309667326328268e-15 -1.9976738756079363e-13
- joint realsense_depth_frame_fixed_joint: origin xyz=0.007515481871156526 0.010000000000000002 1.7352099479506222e-8 rpy=-1.5707963267948966 3.7596758519972983e-16 -1.5707963267948966 -> xyz=0.007415481871156544 0.047499999999999994 1.735209986808428e-8 rpy=-1.5707963267948966 1.439727114483606e-19 -1.570796326794897
- joint realsense_imu_0_fixed_joint: origin xyz=0.007515481871156526 0.010000000000000002 1.7352099479506222e-8 rpy=-1.5707963267948966 3.7596758519972983e-16 -1.5707963267948966 -> xyz=0.007415481871156544 0.047499999999999994 1.735209986808428e-8 rpy=-1.5707963267948966 1.439727114483606e-19 -1.570796326794897
- joint realsense_rgb_frame_fixed_joint: origin xyz=0.007515481871156526 -0.011499999999999996 1.7352099701550827e-8 rpy=-1.5707963267948966 3.7596758519972983e-16 -1.5707963267948966 -> xyz=0.007415481871156544 -0.011499999999999993 1.735209981257313e-8 rpy=-1.5707963267948966 1.439727114483606e-19 -1.570796326794897

File: urdf/ergoCub/robots/ergoCubGazeboSN001_minContacts/model.urdf (robot description, URDF)
Before this commit: robot ergoCub, 205 links, 204 joints
Links:
- link realsense: mass 0.0973042045264468 -> 0.08233251527028056
Joints:
- joint camera_tilt: axis -1.998015835203486e-13 -1 -8.597927048660853e-14 -> -7.529259780358163e-16 -1 -5.660091301660221e-16; origin xyz=0.06250999999999991 -2.999999997621366e-5 0.07639249999999997 rpy=-7.545682259870277e-14 2.5958199361694967e-4 2.017046159162252e-13 -> xyz=0.06250999999999987 -3.000000000113848e-5 0.07639250000000047 rpy=9.528820759122057e-15 2.5958199325913113e-4 2.6559516676797335e-15
- joint l_index_dist: axis -1 -2.9143356888525625e-16 9.714452192336961e-17 -> -1.0000000000000002 -2.359224176539984e-16 1.457167792507203e-16; origin xyz=-2.7755575615628914e-17 -0.0015000000000000013 -0.03999999999999987 rpy=-7.482326172536535e-8 1.8041124150158794e-16 -5.551115123125783e-16 -> xyz=-2.7755575615628914e-17 -0.0014999999999999736 -0.039999999999999925 rpy=-7.482326169760975e-8 1.734723475976807e-16 -5.551115123125782e-16
- joint neck_roll: axis 1 2.30576840860686e-16 -7.196923107658096e-17 -> 1 2.3057684086068286e-16 -7.196923107658096e-17
- joint neck_yaw: axis 1.386477883657293e-15 2.1582026845669262e-16 0.9999999999999999 -> 1.3309667326328268e-15 1.603091172356458e-16 0.9999999999999999; origin xyz=-1.734723475976807e-18 1.0057301276633031e-23 0.06914999999999993 rpy=2.1582026845669264e-16 -1.386477883657293e-15 -1.9981249037222812e-13 -> xyz=-5.0306980803327406e-17 2.0696535769897827e-17 0.06914999999999971 rpy=1.6030911723564583e-16 -1.3309667326328268e-15 -1.9976738756079363e-13
- joint realsense_depth_frame_fixed_joint: origin xyz=0.007515481871156526 0.010000000000000002 1.7352099479506222e-8 rpy=-1.5707963267948966 3.7596758519972983e-16 -1.5707963267948966 -> xyz=0.007415481871156544 0.047499999999999994 1.735209986808428e-8 rpy=-1.5707963267948966 1.439727114483606e-19 -1.570796326794897
- joint realsense_imu_0_fixed_joint: origin xyz=0.007515481871156526 0.010000000000000002 1.7352099479506222e-8 rpy=-1.5707963267948966 3.7596758519972983e-16 -1.5707963267948966 -> xyz=0.007415481871156544 0.047499999999999994 1.735209986808428e-8 rpy=-1.5707963267948966 1.439727114483606e-19 -1.570796326794897
- joint realsense_rgb_frame_fixed_joint: origin xyz=0.007515481871156526 -0.011499999999999996 1.7352099701550827e-8 rpy=-1.5707963267948966 3.7596758519972983e-16 -1.5707963267948966 -> xyz=0.007415481871156544 -0.011499999999999993 1.735209981257313e-8 rpy=-1.5707963267948966 1.439727114483606e-19 -1.570796326794897

File: urdf/ergoCub/robots/ergoCubGazeboSN003/model.urdf (robot description, URDF)
Before this commit: robot ergoCub, 205 links, 204 joints
Links:
- link realsense: mass 0.0973042045264468 -> 0.08233251527028056
Joints:
- joint camera_tilt: axis 2.46237494755185e-16 -1 -1.3590792672083997e-15 -> -7.529259780358055e-16 -1 -5.660091301660095e-16; origin xyz=0.06251000000000004 -3.0000000001050474e-5 0.07639250000000042 rpy=9.111439807333146e-15 2.5958199361708845e-4 1.6567881612289887e-15 -> xyz=0.06250999999999986 -3.0000000001138477e-5 0.07639250000000058 rpy=9.528820759122063e-15 2.595819932592699e-4 2.655951667679724e-15
- joint neck_yaw: axis 1.5706357540212687e-6 5.476218470545924e-15 0.9999999999987664 -> 1.5706357538550546e-6 1.6029881711029372e-16 0.9999999999987664; origin xyz=-1.2588645634161594e-7 -3.511736027695927e-16 0.06914999999990112 rpy=5.476218470552679e-15 -1.5706357540219146e-6 5.308786623366525e-15 -> xyz=-1.2588645629564577e-7 2.1530156161317587e-17 0.06914999999990118 rpy=1.6029881711049145e-16 -1.5706357538557005e-6 1.1347346732224471e-14
- joint realsense_depth_frame_fixed_joint: origin xyz=0.007515481871156526 0.010000000000000002 1.7352099479506222e-8 rpy=-1.5707963267948966 3.7596758519972983e-16 -1.5707963267948966 -> xyz=0.007415481871156544 0.047499999999999994 1.735209986808428e-8 rpy=-1.5707963267948966 1.439727114483606e-19 -1.570796326794897
- joint realsense_imu_0_fixed_joint: origin xyz=0.007515481871156526 0.010000000000000002 1.7352099479506222e-8 rpy=-1.5707963267948966 3.7596758519972983e-16 -1.5707963267948966 -> xyz=0.007415481871156544 0.047499999999999994 1.735209986808428e-8 rpy=-1.5707963267948966 1.439727114483606e-19 -1.570796326794897
- joint realsense_rgb_frame_fixed_joint: origin xyz=0.007515481871156526 -0.011499999999999996 1.7352099701550827e-8 rpy=-1.5707963267948966 3.7596758519972983e-16 -1.5707963267948966 -> xyz=0.007415481871156544 -0.011499999999999993 1.735209981257313e-8 rpy=-1.5707963267948966 1.439727114483606e-19 -1.570796326794897

File: urdf/ergoCub/robots/ergoCubGazeboSN003_minContacts/model.urdf (robot description, URDF)
Before this commit: robot ergoCub, 205 links, 204 joints
Links:
- link realsense: mass 0.0973042045264468 -> 0.08233251527028056
Joints:
- joint camera_tilt: axis 2.46237494755185e-16 -1 -1.3590792672083997e-15 -> -7.529259780358055e-16 -1 -5.660091301660095e-16; origin xyz=0.06251000000000004 -3.0000000001050474e-5 0.07639250000000042 rpy=9.111439807333146e-15 2.5958199361708845e-4 1.6567881612289887e-15 -> xyz=0.06250999999999986 -3.0000000001138477e-5 0.07639250000000058 rpy=9.528820759122063e-15 2.595819932592699e-4 2.655951667679724e-15
- joint neck_yaw: axis 1.5706357540212687e-6 5.476218470545924e-15 0.9999999999987664 -> 1.5706357538550546e-6 1.6029881711029372e-16 0.9999999999987664; origin xyz=-1.2588645634161594e-7 -3.511736027695927e-16 0.06914999999990112 rpy=5.476218470552679e-15 -1.5706357540219146e-6 5.308786623366525e-15 -> xyz=-1.2588645629564577e-7 2.1530156161317587e-17 0.06914999999990118 rpy=1.6029881711049145e-16 -1.5706357538557005e-6 1.1347346732224471e-14
- joint realsense_depth_frame_fixed_joint: origin xyz=0.007515481871156526 0.010000000000000002 1.7352099479506222e-8 rpy=-1.5707963267948966 3.7596758519972983e-16 -1.5707963267948966 -> xyz=0.007415481871156544 0.047499999999999994 1.735209986808428e-8 rpy=-1.5707963267948966 1.439727114483606e-19 -1.570796326794897
- joint realsense_imu_0_fixed_joint: origin xyz=0.007515481871156526 0.010000000000000002 1.7352099479506222e-8 rpy=-1.5707963267948966 3.7596758519972983e-16 -1.5707963267948966 -> xyz=0.007415481871156544 0.047499999999999994 1.735209986808428e-8 rpy=-1.5707963267948966 1.439727114483606e-19 -1.570796326794897
- joint realsense_rgb_frame_fixed_joint: origin xyz=0.007515481871156526 -0.011499999999999996 1.7352099701550827e-8 rpy=-1.5707963267948966 3.7596758519972983e-16 -1.5707963267948966 -> xyz=0.007415481871156544 -0.011499999999999993 1.735209981257313e-8 rpy=-1.5707963267948966 1.439727114483606e-19 -1.570796326794897

File: urdf/ergoCub/robots/ergoCubSN000/model.urdf (robot description, URDF)
Before this commit: robot ergoCub, 204 links, 203 joints
Links:
- link realsense: mass 0.0973042045264468 -> 0.08233251527028056
Joints:
- joint camera_tilt: axis 1.9074075506529947e-16 -1 -1.4146048262463281e-15 -> -7.529259780358045e-16 -1 -5.660091301660127e-16; origin xyz=0.06251 -3.0000000001127547e-5 0.0763925000000007 rpy=9.055928654249867e-15 2.5958199361703294e-4 1.7122849027886369e-15 -> xyz=0.06250999999999989 -3.0000000001138484e-5 0.07639250000000042 rpy=9.528820759122059e-15 2.595819932592144e-4 2.6559516676797224e-15
- joint l_index_dist: axis -0.9999999999999997 1.2698175844150033e-15 1.3045120539345794e-15 -> -0.9999999999999999 1.3253287356462613e-15 1.2351231148955076e-15; origin xyz=4.163336342344337e-17 -0.0015000000000000013 -0.030000000000000082 rpy=-1.6320278461989814e-14 -1.1102230246251565e-16 1.110223024625157e-16 -> xyz=2.7755575615628914e-17 -0.0015000000000000568 -0.02999999999999997 rpy=-1.6320278461989807e-14 -5.551115123125783e-17 5.551115123125784e-17
- joint l_index_prox: axis -0.9999999999999996 -2.0816681711721439e-16 3.99680288865056e-15 -> -0.9999999999999998 -2.0816681711721453e-16 3.996802888650561e-15; origin xyz=0.009192533317427712 -2.7755575615628914e-17 -0.030713451316238316 rpy=6.383782391594655e-16 -1.942890293094024e-16 1.110223024625157e-16 -> xyz=0.00919253331742774 0 -0.030713451316238427 rpy=6.106226635438364e-16 -2.636779683484747e-16 5.551115123125784e-17
- joint neck_yaw: axis 1.4082090529075477e-15 5.709519748275242e-16 0.9999999999999998 -> 1.6591628191298083e-15 5.987076998014226e-16 0.9999999999999998; origin xyz=-1.3010426069826053e-17 3.765597982987134e-17 0.0691500000000001 rpy=1.9500353504997633e-16 -1.4141248935670295e-15 3.767470613092508e-16 -> xyz=-4.0766001685454967e-17 3.151498988337666e-17 0.0691500000000001 rpy=2.2275926002387476e-16 -1.6650786597892902e-15 3.2676263100504264e-16
- joint realsense_depth_frame_fixed_joint: origin xyz=0.007515481871156526 0.010000000000000002 1.7352099479506222e-8 rpy=-1.5707963267948966 3.7596758519972983e-16 -1.5707963267948966 -> xyz=0.007415481871156544 0.047499999999999994 1.735209986808428e-8 rpy=-1.5707963267948966 1.439727114483606e-19 -1.570796326794897
- joint realsense_imu_0_fixed_joint: origin xyz=0.007515481871156526 0.010000000000000002 1.7352099479506222e-8 rpy=-1.5707963267948966 3.7596758519972983e-16 -1.5707963267948966 -> xyz=0.007415481871156544 0.047499999999999994 1.735209986808428e-8 rpy=-1.5707963267948966 1.439727114483606e-19 -1.570796326794897
- joint realsense_rgb_frame_fixed_joint: origin xyz=0.007515481871156526 -0.011499999999999996 1.7352099701550827e-8 rpy=-1.5707963267948966 3.7596758519972983e-16 -1.5707963267948966 -> xyz=0.007415481871156544 -0.011499999999999993 1.735209981257313e-8 rpy=-1.5707963267948966 1.439727114483606e-19 -1.570796326794897

File: urdf/ergoCub/robots/ergoCubSN001/model.urdf (robot description, URDF)
Before this commit: robot ergoCub, 205 links, 204 joints
Links:
- link realsense: mass 0.0973042045264468 -> 0.08233251527028056
Joints:
- joint camera_tilt: axis -1.998015835203486e-13 -1 -8.597927048660853e-14 -> -7.529259780358163e-16 -1 -5.660091301660221e-16; origin xyz=0.06250999999999991 -2.999999997621366e-5 0.07639249999999997 rpy=-7.545682259870277e-14 2.5958199361694967e-4 2.017046159162252e-13 -> xyz=0.06250999999999987 -3.000000000113848e-5 0.07639250000000047 rpy=9.528820759122057e-15 2.5958199325913113e-4 2.6559516676797335e-15
- joint l_index_dist: axis -1 -2.9143356888525625e-16 9.714452192336961e-17 -> -1.0000000000000002 -2.359224176539984e-16 1.457167792507203e-16; origin xyz=-2.7755575615628914e-17 -0.0015000000000000013 -0.03999999999999987 rpy=-7.482326172536535e-8 1.8041124150158794e-16 -5.551115123125783e-16 -> xyz=-2.7755575615628914e-17 -0.0014999999999999736 -0.039999999999999925 rpy=-7.482326169760975e-8 1.734723475976807e-16 -5.551115123125782e-16
- joint neck_roll: axis 1 2.30576840860686e-16 -7.196923107658096e-17 -> 1 2.3057684086068286e-16 -7.196923107658096e-17
- joint neck_yaw: axis 1.386477883657293e-15 2.1582026845669262e-16 0.9999999999999999 -> 1.3309667326328268e-15 1.603091172356458e-16 0.9999999999999999; origin xyz=-1.734723475976807e-18 1.0057301276633031e-23 0.06914999999999993 rpy=2.1582026845669264e-16 -1.386477883657293e-15 -1.9981249037222812e-13 -> xyz=-5.0306980803327406e-17 2.0696535769897827e-17 0.06914999999999971 rpy=1.6030911723564583e-16 -1.3309667326328268e-15 -1.9976738756079363e-13
- joint realsense_depth_frame_fixed_joint: origin xyz=0.007515481871156526 0.010000000000000002 1.7352099479506222e-8 rpy=-1.5707963267948966 3.7596758519972983e-16 -1.5707963267948966 -> xyz=0.007415481871156544 0.047499999999999994 1.735209986808428e-8 rpy=-1.5707963267948966 1.439727114483606e-19 -1.570796326794897
- joint realsense_imu_0_fixed_joint: origin xyz=0.007515481871156526 0.010000000000000002 1.7352099479506222e-8 rpy=-1.5707963267948966 3.7596758519972983e-16 -1.5707963267948966 -> xyz=0.007415481871156544 0.047499999999999994 1.735209986808428e-8 rpy=-1.5707963267948966 1.439727114483606e-19 -1.570796326794897
- joint realsense_rgb_frame_fixed_joint: origin xyz=0.007515481871156526 -0.011499999999999996 1.7352099701550827e-8 rpy=-1.5707963267948966 3.7596758519972983e-16 -1.5707963267948966 -> xyz=0.007415481871156544 -0.011499999999999993 1.735209981257313e-8 rpy=-1.5707963267948966 1.439727114483606e-19 -1.570796326794897

File: urdf/ergoCub/robots/ergoCubSN003/model.urdf (robot description, URDF)
Before this commit: robot ergoCub, 205 links, 204 joints
Links:
- link realsense: mass 0.0973042045264468 -> 0.08233251527028056
Joints:
- joint camera_tilt: axis 2.46237494755185e-16 -1 -1.3590792672083997e-15 -> -7.529259780358055e-16 -1 -5.660091301660095e-16; origin xyz=0.06251000000000004 -3.0000000001050474e-5 0.07639250000000042 rpy=9.111439807333146e-15 2.5958199361708845e-4 1.6567881612289887e-15 -> xyz=0.06250999999999986 -3.0000000001138477e-5 0.07639250000000058 rpy=9.528820759122063e-15 2.595819932592699e-4 2.655951667679724e-15
- joint neck_yaw: axis 1.5706357540212687e-6 5.476218470545924e-15 0.9999999999987664 -> 1.5706357538550546e-6 1.6029881711029372e-16 0.9999999999987664; origin xyz=-1.2588645634161594e-7 -3.511736027695927e-16 0.06914999999990112 rpy=5.476218470552679e-15 -1.5706357540219146e-6 5.308786623366525e-15 -> xyz=-1.2588645629564577e-7 2.1530156161317587e-17 0.06914999999990118 rpy=1.6029881711049145e-16 -1.5706357538557005e-6 1.1347346732224471e-14
- joint realsense_depth_frame_fixed_joint: origin xyz=0.007515481871156526 0.010000000000000002 1.7352099479506222e-8 rpy=-1.5707963267948966 3.7596758519972983e-16 -1.5707963267948966 -> xyz=0.007415481871156544 0.047499999999999994 1.735209986808428e-8 rpy=-1.5707963267948966 1.439727114483606e-19 -1.570796326794897
- joint realsense_imu_0_fixed_joint: origin xyz=0.007515481871156526 0.010000000000000002 1.7352099479506222e-8 rpy=-1.5707963267948966 3.7596758519972983e-16 -1.5707963267948966 -> xyz=0.007415481871156544 0.047499999999999994 1.735209986808428e-8 rpy=-1.5707963267948966 1.439727114483606e-19 -1.570796326794897
- joint realsense_rgb_frame_fixed_joint: origin xyz=0.007515481871156526 -0.011499999999999996 1.7352099701550827e-8 rpy=-1.5707963267948966 3.7596758519972983e-16 -1.5707963267948966 -> xyz=0.007415481871156544 -0.011499999999999993 1.735209981257313e-8 rpy=-1.5707963267948966 1.439727114483606e-19 -1.570796326794897
